File: examples/generated/kicad/bjt_common_emitter.kicad_sch (KiCad schematic)
At the start: 6 parts, among them Q1 2N3904

Commit message: Generate schematics that are more intelligible and project structure that is closer to the KiCad demo behavior.
Other:
- note added: "pins 1:collector 2:base 3:emitter"
- note added: "pins 1:emitter 2:0"
- note added: "pins 1:vcc 2:0"
- note added: "pins 1:vcc 2:base"
- note added: "pins 1:vcc 2:collector"
- note added: "pins 1:vin 2:0"
Changed lines of the file:
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@@
     (effects (font (size 1.27 1.27)) (justify left))
+  )
+  (text "pins 1:vcc  2:0" (at 50 58 0)
+    (effects (font (size 1.0 1.0)) (justify left))
   )
   (symbol (lib_id "pspice:VSOURCE") (at 50 50 0) (unit 1)
@@
     (effects (font (size 1.27 1.27)) (justify left))
   )
+  (text "pins 1:vin  2:0" (at 85 58 0)
+    (effects (font (size 1.0 1.0)) (justify left))
+  )
   (symbol (lib_id "pspice:VSOURCE") (at 85 50 0) (unit 1)
     (in_bom yes) (on_board yes)
@@
   (text "nodes: vcc base" (at 120 42 0)
     (effects (font (size 1.27 1.27)) (justify left))
+  )
+  (text "pins 1:vcc  2:base" (at 120 58 0)
+    (effects (font (size 1.0 1.0)) (justify left))
   )
   (symbol (lib_id "Device:R") (at 120 50 0) (unit 1)
@@
     (effects (font (size 1.27 1.27)) (justify left))
   )
+  (text "pins 1:vcc  2:collector" (at 155 58 0)
+    (effects (font (size 1.0 1.0)) (justify left))
+  )
   (symbol (lib_id "Device:R") (at 155 50 0) (unit 1)
     (in_bom yes) (on_board yes)
@@
   (text "nodes: emitter 0" (at 50 72 0)
     (effects (font (size 1.27 1.27)) (justify left))
+  )
+  (text "pins 1:emitter  2:0" (at 50 88 0)
+    (effects (font (size 1.0 1.0)) (justify left))
   )
   (symbol (lib_id "Device:R") (at 50 80 0) (unit 1)
@@
     (effects (font (size 1.27 1.27)) (justify left))
   )
+  (text "pins 1:collector  2:base  3:emitter" (at 85 88 0)
+    (effects (font (size 1.0 1.0)) (justify left))
+  )
   (symbol (lib_id "Device:Q_NPN_BCE") (at 85 80 0) (unit 1)

Commit message: Attempt to clean up symbols and schematics to be more himan readable.
Other:
- note removed: "nodes: collector base emitter"
- note removed: "nodes: emitter 0"
- note removed: "nodes: vcc 0"
- note removed: "nodes: vcc base"
- note removed: "nodes: vcc collector"
- note removed: "nodes: vin 0"
- note removed: "pins 1:collector 2:base 3:emitter"
- note removed: "pins 1:emitter 2:0"
- note removed: "pins 1:vcc 2:0"
- note removed: "pins 1:vcc 2:base"
- note removed: "pins 1:vcc 2:collector"
- note removed: "pins 1:vin 2:0"
- title: (none) -> bjt_common_emitter
Changed lines of the file:
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@@
   (generator "mixedsig2cad")
   (paper "A4")
-  (text "nodes: vcc 0" (at 50 42 0)
-    (effects (font (size 1.27 1.27)) (justify left))
-  )
-  (text "pins 1:vcc  2:0" (at 50 58 0)
-    (effects (font (size 1.0 1.0)) (justify left))
+  (title_block
+    (title "bjt_common_emitter")
+    (date "2026-03-05")
+    (comment 1 "Generated by mixedsig2cad")
   )
   (symbol (lib_id "pspice:VSOURCE") (at 50 50 0) (unit 1)
@@
     )
   )
-  (text "nodes: vin 0" (at 85 42 0)
-    (effects (font (size 1.27 1.27)) (justify left))
-  )
-  (text "pins 1:vin  2:0" (at 85 58 0)
-    (effects (font (size 1.0 1.0)) (justify left))
-  )
   (symbol (lib_id "pspice:VSOURCE") (at 85 50 0) (unit 1)
     (in_bom yes) (on_board yes)
@@
       (effects (font (size 1.27 1.27)) hide)
     )
-  )
-  (text "nodes: vcc base" (at 120 42 0)
-    (effects (font (size 1.27 1.27)) (justify left))
-  )
-  (text "pins 1:vcc  2:base" (at 120 58 0)
-    (effects (font (size 1.0 1.0)) (justify left))
   )
   (symbol (lib_id "Device:R") (at 120 50 0) (unit 1)
@@
     )
   )
-  (text "nodes: vcc collector" (at 155 42 0)
-    (effects (font (size 1.27 1.27)) (justify left))
-  )
-  (text "pins 1:vcc  2:collector" (at 155 58 0)
-    (effects (font (size 1.0 1.0)) (justify left))
-  )
   (symbol (lib_id "Device:R") (at 155 50 0) (unit 1)
     (in_bom yes) (on_board yes)
@@
       (effects (font (size 1.27 1.27)) hide)
     )
-  )
-  (text "nodes: emitter 0" (at 50 72 0)
-    (effects (font (size 1.27 1.27)) (justify left))
-  )
-  (text "pins 1:emitter  2:0" (at 50 88 0)
-    (effects (font (size 1.0 1.0)) (justify left))
   )
   (symbol (lib_id "Device:R") (at 50 80 0) (unit 1)
@@
     )
   )
-  (text "nodes: collector base emitter" (at 85 72 0)
-    (effects (font (size 1.27 1.27)) (justify left))
-  )
-  (text "pins 1:collector  2:base  3:emitter" (at 85 88 0)
-    (effects (font (size 1.0 1.0)) (justify left))
-  )
   (symbol (lib_id "Device:Q_NPN_BCE") (at 85 80 0) (unit 1)
     (in_bom yes) (on_board yes)
@@
     )
   )
+  (label "0" (at 50.00 54.50 0)
+    (effects (font (size 1.27 1.27)) (justify left bottom))
+  )
+  (wire (pts (xy 55.00 72.00) (xy 92.00 72.00))
+    (stroke (width 0) (type solid) (color 0 0 0 0))
+  )
+  (wire (pts (xy 56.00 56.00) (xy 56.00 72.00))
+    (stroke (width 0) (type solid) (color 0 0 0 0))
+  )
+  (junction (at 56.00 72.00) (diameter 1.016) (color 0 0 0 0))
+  (wire (pts (xy 91.00 56.00) (xy 91.00 72.00))
+    (stroke (width 0) (type solid) (color 0 0 0 0))
+  )
+  (junction (at 91.00 72.00) (diameter 1.016) (color 0 0 0 0))
+  (wire (pts (xy 56.00 86.00) (xy 56.00 72.00))
+    (stroke (width 0) (type solid) (color 0 0 0 0))
+  )
+  (junction (at 56.00 72.00) (diameter 1.016) (color 0 0 0 0))
+  (label "base" (at 79.00 53.00 0)
+    (effects (font (size 1.27 1.27)) (justify left bottom))
+  )
+  (wire (pts (xy 126.00 56.00) (xy 105.50 56.00))
+    (stroke (width 0) (type solid) (color 0 0 0 0))
+  )
+  (wire (pts (xy 105.50 56.00) (xy 105.50 74.00))
+    (stroke (width 0) (type solid) (color 0 0 0 0))
+  )
+  (wire (pts (xy 105.50 74.00) (xy 85.00 74.00))
+    (stroke (width 0) (type solid) (color 0 0 0 0))
+  )
+  (junction (at 105.50 56.00) (diameter 1.016) (color 0 0 0 0))
+  (junction (at 105.50 74.00) (diameter 1.016) (color 0 0 0 0))
+  (label "collector" (at 73.00 54.50 0)
+    (effects (font (size 1.27 1.27)) (justify left bottom))
+  )
+  (wire (pts (xy 161.00 56.00) (xy 120.00 56.00))
+    (stroke (width 0) (type solid) (color 0 0 0 0))
+  )
+  (wire (pts (xy 120.00 56.00) (xy 120.00 74.00))
+    (stroke (width 0) (type solid) (color 0 0 0 0))
+  )
+  (wire (pts (xy 120.00 74.00) (xy 79.00 74.00))
+    (stroke (width 0) (type solid) (color 0 0 0 0))
+  )
+  (junction (at 120.00 56.00) (diameter 1.016) (color 0 0 0 0))
+  (junction (at 120.00 74.00) (diameter 1.016) (color 0 0 0 0))
+  (label "emitter" (at 38.00 71.00 0)
+    (effects (font (size 1.27 1.27)) (justify left bottom))
+  )
+  (wire (pts (xy 44.00 74.00) (xy 67.50 74.00))
+    (stroke (width 0) (type solid) (color 0 0 0 0))
+  )
+  (wire (pts (xy 67.50 74.00) (xy 67.50 86.00))
+    (stroke (width 0) (type solid) (color 0 0 0 0))
+  )
+  (wire (pts (xy 67.50 86.00) (xy 91.00 86.00))
+    (stroke (width 0) (type solid) (color 0 0 0 0))
+  )
+  (junction (at 67.50 74.00) (diameter 1.016) (color 0 0 0 0))
+  (junction (at 67.50 86.00) (diameter 1.016) (color 0 0 0 0))
+  (label "vcc" (at 38.00 42.50 0)
+    (effects (font (size 1.27 1.27)) (justify left bottom))
+  )
+  (wire (pts (xy 43.00 50.00) (xy 150.00 50.00))
+    (stroke (width 0) (type solid) (color 0 0 0 0))
+  )
+  (wire (pts (xy 44.00 44.00) (xy 44.00 50.00))
+    (stroke (width 0) (type solid) (color 0 0 0 0))
+  )
+  (junction (at 44.00 50.00) (diameter 1.016) (color 0 0 0 0))
+  (wire (pts (xy 114.00 44.00) (xy 114.00 50.00))
+    (stroke (width 0) (type solid) (color 0 0 0 0))
+  )
+  (junction (at 114.00 50.00) (diameter 1.016) (color 0 0 0 0))
+  (wire (pts (xy 149.00 44.00) (xy 149.00 50.00))
+    (stroke (width 0) (type solid) (color 0 0 0 0))
+  )
+  (junction (at 149.00 50.00) (diameter 1.016) (color 0 0 0 0))
+  (label "vin" (at 73.00 41.00 0)
+    (effects (font (size 1.27 1.27)) (justify left bottom))
+  )
   (sheet_instances

Commit message: Attempt to add power symbology.
Parts:
- Q1: symbol Device:Q_NPN_BCE -> examples:QNPN
- RB, RC, RE: symbol Device:R -> examples:R
- VCC, VIN: symbol pspice:VSOURCE -> examples:VSOURCE
Changed lines of the file:
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@@
     (comment 1 "Generated by mixedsig2cad")
   )
-  (symbol (lib_id "pspice:VSOURCE") (at 50 50 0) (unit 1)
+  (symbol (lib_id "examples:VSOURCE") (at 50 50 0) (unit 1)
     (in_bom yes) (on_board yes)
     (property "Reference" "VCC" (at 50 46.19 0)
@@
     )
   )
-  (symbol (lib_id "pspice:VSOURCE") (at 85 50 0) (unit 1)
+  (symbol (lib_id "examples:VSOURCE") (at 85 50 0) (unit 1)
     (in_bom yes) (on_board yes)
     (property "Reference" "VIN" (at 85 46.19 0)
@@
     )
   )
-  (symbol (lib_id "Device:R") (at 120 50 0) (unit 1)
+  (symbol (lib_id "examples:R") (at 120 50 0) (unit 1)
     (in_bom yes) (on_board yes)
     (property "Reference" "RB" (at 120 46.19 0)
@@
     )
   )
-  (symbol (lib_id "Device:R") (at 155 50 0) (unit 1)
+  (symbol (lib_id "examples:R") (at 155 50 0) (unit 1)
     (in_bom yes) (on_board yes)
     (property "Reference" "RC" (at 155 46.19 0)
@@
     )
   )
-  (symbol (lib_id "Device:R") (at 50 80 0) (unit 1)
+  (symbol (lib_id "examples:R") (at 50 80 0) (unit 1)
     (in_bom yes) (on_board yes)
     (property "Reference" "RE" (at 50 76.19 0)
@@
     )
   )
-  (symbol (lib_id "Device:Q_NPN_BCE") (at 85 80 0) (unit 1)
+  (symbol (lib_id "examples:QNPN") (at 85 80 0) (unit 1)
     (in_bom yes) (on_board yes)
     (property "Reference" "Q1" (at 85 76.19 0)
@@
     )
   )
-  (label "0" (at 50.00 54.50 0)
-    (effects (font (size 1.27 1.27)) (justify left bottom))
-  )
-  (wire (pts (xy 55.00 72.00) (xy 92.00 72.00))
-    (stroke (width 0) (type solid) (color 0 0 0 0))
-  )
-  (wire (pts (xy 56.00 56.00) (xy 56.00 72.00))
-    (stroke (width 0) (type solid) (color 0 0 0 0))
-  )
-  (junction (at 56.00 72.00) (diameter 1.016) (color 0 0 0 0))
-  (wire (pts (xy 91.00 56.00) (xy 91.00 72.00))
-    (stroke (width 0) (type solid) (color 0 0 0 0))
-  )
-  (junction (at 91.00 72.00) (diameter 1.016) (color 0 0 0 0))
-  (wire (pts (xy 56.00 86.00) (xy 56.00 72.00))
-    (stroke (width 0) (type solid) (color 0 0 0 0))
-  )
-  (junction (at 56.00 72.00) (diameter 1.016) (color 0 0 0 0))
+  (symbol (lib_id "examples:GND") (at 44.00 50.00 0) (unit 1)
+    (in_bom yes) (on_board yes)
+    (property "Reference" "#PWR0001" (at 44.0 46.19 0)
+      (effects (font (size 1.27 1.27)) hide)
+    )
+    (property "Value" "GND" (at 44.0 53.81 0)
+      (effects (font (size 1.27 1.27)))
+    )
+    (property "Footprint" "" (at 0 0 0)
+      (effects (font (size 1.27 1.27)) hide)
+    )
+    (property "Datasheet" "" (at 0 0 0)
+      (effects (font (size 1.27 1.27)) hide)
+    )
+  )
+  (symbol (lib_id "examples:VCC") (at 32.00 38.00 0) (unit 1)
+    (in_bom yes) (on_board yes)
+    (property "Reference" "#PWR0002" (at 32.0 34.19 0)
+      (effects (font (size 1.27 1.27)) hide)
+    )
+    (property "Value" "VCC" (at 32.0 41.81 0)
+      (effects (font (size 1.27 1.27)))
+    )
+    (property "Footprint" "" (at 0 0 0)
+      (effects (font (size 1.27 1.27)) hide)
+    )
+    (property "Datasheet" "" (at 0 0 0)
+      (effects (font (size 1.27 1.27)) hide)
+    )
+  )
+  (label "GND" (at 38.00 48.50 0)
+    (effects (font (size 1.27 1.27)) (justify left bottom))
+  )
+  (wire (pts (xy 43.00 68.00) (xy 92.00 68.00))
+    (stroke (width 0) (type solid) (color 0 0 0 0))
+  )
+  (wire (pts (xy 56.00 56.00) (xy 56.00 68.00))
+    (stroke (width 0) (type solid) (color 0 0 0 0))
+  )
+  (junction (at 56.00 68.00) (diameter 1.016) (color 0 0 0 0))
+  (wire (pts (xy 91.00 56.00) (xy 91.00 68.00))
+    (stroke (width 0) (type solid) (color 0 0 0 0))
+  )
+  (junction (at 91.00 68.00) (diameter 1.016) (color 0 0 0 0))
+  (wire (pts (xy 56.00 86.00) (xy 56.00 68.00))
+    (stroke (width 0) (type solid) (color 0 0 0 0))
+  )
+  (junction (at 56.00 68.00) (diameter 1.016) (color 0 0 0 0))
+  (wire (pts (xy 44.00 50.00) (xy 44.00 68.00))
+    (stroke (width 0) (type solid) (color 0 0 0 0))
+  )
+  (junction (at 44.00 68.00) (diameter 1.016) (color 0 0 0 0))
   (label "base" (at 79.00 53.00 0)
     (effects (font (size 1.27 1.27)) (justify left bottom))
@@
   (junction (at 67.50 74.00) (diameter 1.016) (color 0 0 0 0))
   (junction (at 67.50 86.00) (diameter 1.016) (color 0 0 0 0))
-  (label "vcc" (at 38.00 42.50 0)
-    (effects (font (size 1.27 1.27)) (justify left bottom))
-  )
-  (wire (pts (xy 43.00 50.00) (xy 150.00 50.00))
-    (stroke (width 0) (type solid) (color 0 0 0 0))
-  )
-  (wire (pts (xy 44.00 44.00) (xy 44.00 50.00))
-    (stroke (width 0) (type solid) (color 0 0 0 0))
-  )
-  (junction (at 44.00 50.00) (diameter 1.016) (color 0 0 0 0))
-  (wire (pts (xy 114.00 44.00) (xy 114.00 50.00))
-    (stroke (width 0) (type solid) (color 0 0 0 0))
-  )
-  (junction (at 114.00 50.00) (diameter 1.016) (color 0 0 0 0))
-  (wire (pts (xy 149.00 44.00) (xy 149.00 50.00))
-    (stroke (width 0) (type solid) (color 0 0 0 0))
-  )
-  (junction (at 149.00 50.00) (diameter 1.016) (color 0 0 0 0))
+  (label "VCC" (at 26.00 36.50 0)
+    (effects (font (size 1.27 1.27)) (justify left bottom))
+  )
+  (wire (pts (xy 31.00 48.50) (xy 150.00 48.50))
+    (stroke (width 0) (type solid) (color 0 0 0 0))
+  )
+  (wire (pts (xy 44.00 44.00) (xy 44.00 48.50))
+    (stroke (width 0) (type solid) (color 0 0 0 0))
+  )
+  (junction (at 44.00 48.50) (diameter 1.016) (color 0 0 0 0))
+  (wire (pts (xy 114.00 44.00) (xy 114.00 48.50))
+    (stroke (width 0) (type solid) (color 0 0 0 0))
+  )
+  (junction (at 114.00 48.50) (diameter 1.016) (color 0 0 0 0))
+  (wire (pts (xy 149.00 44.00) (xy 149.00 48.50))
+    (stroke (width 0) (type solid) (color 0 0 0 0))
+  )
+  (junction (at 149.00 48.50) (diameter 1.016) (color 0 0 0 0))
+  (wire (pts (xy 32.00 38.00) (xy 32.00 48.50))
+    (stroke (width 0) (type solid) (color 0 0 0 0))
+  )
+  (junction (at 32.00 48.50) (diameter 1.016) (color 0 0 0 0))
   (label "vin" (at 73.00 41.00 0)
     (effects (font (size 1.27 1.27)) (justify left bottom))
@@
     (path "/700fe220-286d-536e-b5fd-6550242a4c6e" (reference "RE") (unit 1) (value "1k") (footprint ""))
     (path "/88a76c4e-b40d-5bca-899e-ae1b281ceeb7" (reference "Q1") (unit 1) (value "2N3904") (footprint ""))
+    (path "/5a029890-81cb-5adb-a892-c4ff0d7135d4" (reference "#PWR0001") (unit 1) (value "GND") (footprint ""))
+    (path "/59a1f20f-d5c2-5035-b859-86ff53683043" (reference "#PWR0002") (unit 1) (value "VCC") (footprint ""))
   )
 )
