File: examples/generated/kicad/cmos_inverter.kicad_sch (KiCad schematic)
At the start: 4 parts

Commit message: Generate schematics that are more intelligible and project structure that is closer to the KiCad demo behavior.
Parts:
- MN1: symbol Device:Q_PMOS_GSD -> Device:Q_NMOS_GSD
Other:
- note added: "pins 1:vdd 2:0"
- note added: "pins 1:vin 2:0"
- note added: "pins 1:vout 2:vin 3:0 4:0"
- note added: "pins 1:vout 2:vin 3:vdd 4:vdd"
Changed lines of the file:
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@@
     (effects (font (size 1.27 1.27)) (justify left))
+  )
+  (text "pins 1:vdd  2:0" (at 50 58 0)
+    (effects (font (size 1.0 1.0)) (justify left))
   )
   (symbol (lib_id "pspice:VSOURCE") (at 50 50 0) (unit 1)
@@
     (effects (font (size 1.27 1.27)) (justify left))
   )
+  (text "pins 1:vin  2:0" (at 85 58 0)
+    (effects (font (size 1.0 1.0)) (justify left))
+  )
   (symbol (lib_id "pspice:VSOURCE") (at 85 50 0) (unit 1)
     (in_bom yes) (on_board yes)
@@
   (text "nodes: vout vin vdd vdd" (at 120 42 0)
     (effects (font (size 1.27 1.27)) (justify left))
+  )
+  (text "pins 1:vout  2:vin  3:vdd  4:vdd" (at 120 58 0)
+    (effects (font (size 1.0 1.0)) (justify left))
   )
   (symbol (lib_id "Device:Q_PMOS_GSD") (at 120 50 0) (unit 1)
@@
     (effects (font (size 1.27 1.27)) (justify left))
   )
-  (symbol (lib_id "Device:Q_PMOS_GSD") (at 155 50 0) (unit 1)
+  (text "pins 1:vout  2:vin  3:0  4:0" (at 155 58 0)
+    (effects (font (size 1.0 1.0)) (justify left))
+  )
+  (symbol (lib_id "Device:Q_NMOS_GSD") (at 155 50 0) (unit 1)
     (in_bom yes) (on_board yes)
     (property "Reference" "MN1" (at 155 46.19 0)

Commit message: Attempt to clean up symbols and schematics to be more himan readable.
Other:
- note removed: "nodes: vdd 0"
- note removed: "nodes: vin 0"
- note removed: "nodes: vout vin 0 0"
- note removed: "nodes: vout vin vdd vdd"
- note removed: "pins 1:vdd 2:0"
- note removed: "pins 1:vin 2:0"
- note removed: "pins 1:vout 2:vin 3:0 4:0"
- note removed: "pins 1:vout 2:vin 3:vdd 4:vdd"
- title: (none) -> cmos_inverter
Changed lines of the file:
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@@
   (generator "mixedsig2cad")
   (paper "A4")
-  (text "nodes: vdd 0" (at 50 42 0)
-    (effects (font (size 1.27 1.27)) (justify left))
-  )
-  (text "pins 1:vdd  2:0" (at 50 58 0)
-    (effects (font (size 1.0 1.0)) (justify left))
+  (title_block
+    (title "cmos_inverter")
+    (date "2026-03-05")
+    (comment 1 "Generated by mixedsig2cad")
   )
   (symbol (lib_id "pspice:VSOURCE") (at 50 50 0) (unit 1)
@@
     )
   )
-  (text "nodes: vin 0" (at 85 42 0)
-    (effects (font (size 1.27 1.27)) (justify left))
-  )
-  (text "pins 1:vin  2:0" (at 85 58 0)
-    (effects (font (size 1.0 1.0)) (justify left))
-  )
   (symbol (lib_id "pspice:VSOURCE") (at 85 50 0) (unit 1)
     (in_bom yes) (on_board yes)
@@
       (effects (font (size 1.27 1.27)) hide)
     )
-  )
-  (text "nodes: vout vin vdd vdd" (at 120 42 0)
-    (effects (font (size 1.27 1.27)) (justify left))
-  )
-  (text "pins 1:vout  2:vin  3:vdd  4:vdd" (at 120 58 0)
-    (effects (font (size 1.0 1.0)) (justify left))
   )
   (symbol (lib_id "Device:Q_PMOS_GSD") (at 120 50 0) (unit 1)
@@
     )
   )
-  (text "nodes: vout vin 0 0" (at 155 42 0)
-    (effects (font (size 1.27 1.27)) (justify left))
-  )
-  (text "pins 1:vout  2:vin  3:0  4:0" (at 155 58 0)
-    (effects (font (size 1.0 1.0)) (justify left))
-  )
   (symbol (lib_id "Device:Q_NMOS_GSD") (at 155 50 0) (unit 1)
     (in_bom yes) (on_board yes)
@@
     )
   )
+  (label "0" (at 50.00 54.50 0)
+    (effects (font (size 1.27 1.27)) (justify left bottom))
+  )
+  (wire (pts (xy 55.00 62.00) (xy 162.00 62.00))
+    (stroke (width 0) (type solid) (color 0 0 0 0))
+  )
+  (wire (pts (xy 56.00 56.00) (xy 56.00 62.00))
+    (stroke (width 0) (type solid) (color 0 0 0 0))
+  )
+  (junction (at 56.00 62.00) (diameter 1.016) (color 0 0 0 0))
+  (wire (pts (xy 91.00 56.00) (xy 91.00 62.00))
+    (stroke (width 0) (type solid) (color 0 0 0 0))
+  )
+  (junction (at 91.00 62.00) (diameter 1.016) (color 0 0 0 0))
+  (wire (pts (xy 157.00 56.00) (xy 157.00 62.00))
+    (stroke (width 0) (type solid) (color 0 0 0 0))
+  )
+  (junction (at 157.00 62.00) (diameter 1.016) (color 0 0 0 0))
+  (wire (pts (xy 161.00 56.00) (xy 161.00 62.00))
+    (stroke (width 0) (type solid) (color 0 0 0 0))
+  )
+  (junction (at 161.00 62.00) (diameter 1.016) (color 0 0 0 0))
+  (label "vdd" (at 38.00 41.00 0)
+    (effects (font (size 1.27 1.27)) (justify left bottom))
+  )
+  (wire (pts (xy 43.00 58.00) (xy 127.00 58.00))
+    (stroke (width 0) (type solid) (color 0 0 0 0))
+  )
+  (wire (pts (xy 44.00 44.00) (xy 44.00 58.00))
+    (stroke (width 0) (type solid) (color 0 0 0 0))
+  )
+  (junction (at 44.00 58.00) (diameter 1.016) (color 0 0 0 0))
+  (wire (pts (xy 122.00 56.00) (xy 122.00 58.00))
+    (stroke (width 0) (type solid) (color 0 0 0 0))
+  )
+  (junction (at 122.00 58.00) (diameter 1.016) (color 0 0 0 0))
+  (wire (pts (xy 126.00 56.00) (xy 126.00 58.00))
+    (stroke (width 0) (type solid) (color 0 0 0 0))
+  )
+  (junction (at 126.00 58.00) (diameter 1.016) (color 0 0 0 0))
+  (label "vin" (at 73.00 42.50 0)
+    (effects (font (size 1.27 1.27)) (justify left bottom))
+  )
+  (wire (pts (xy 78.00 50.00) (xy 154.00 50.00))
+    (stroke (width 0) (type solid) (color 0 0 0 0))
+  )
+  (wire (pts (xy 79.00 44.00) (xy 79.00 50.00))
+    (stroke (width 0) (type solid) (color 0 0 0 0))
+  )
+  (junction (at 79.00 50.00) (diameter 1.016) (color 0 0 0 0))
+  (wire (pts (xy 118.00 44.00) (xy 118.00 50.00))
+    (stroke (width 0) (type solid) (color 0 0 0 0))
+  )
+  (junction (at 118.00 50.00) (diameter 1.016) (color 0 0 0 0))
+  (wire (pts (xy 153.00 44.00) (xy 153.00 50.00))
+    (stroke (width 0) (type solid) (color 0 0 0 0))
+  )
+  (junction (at 153.00 50.00) (diameter 1.016) (color 0 0 0 0))
+  (label "vout" (at 108.00 41.00 0)
+    (effects (font (size 1.27 1.27)) (justify left bottom))
+  )
+  (wire (pts (xy 114.00 44.00) (xy 149.00 44.00))
+    (stroke (width 0) (type solid) (color 0 0 0 0))
+  )
   (sheet_instances

Commit message: Attempt to add power symbology.
Parts:
- MN1: symbol Device:Q_NMOS_GSD -> examples:MNMOS
- MP1: symbol Device:Q_PMOS_GSD -> examples:MPMOS
- VDD, VIN: symbol pspice:VSOURCE -> examples:VSOURCE
Changed lines of the file:
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@@
     (comment 1 "Generated by mixedsig2cad")
   )
-  (symbol (lib_id "pspice:VSOURCE") (at 50 50 0) (unit 1)
+  (symbol (lib_id "examples:VSOURCE") (at 50 50 0) (unit 1)
     (in_bom yes) (on_board yes)
     (property "Reference" "VDD" (at 50 46.19 0)
@@
     )
   )
-  (symbol (lib_id "pspice:VSOURCE") (at 85 50 0) (unit 1)
+  (symbol (lib_id "examples:VSOURCE") (at 85 50 0) (unit 1)
     (in_bom yes) (on_board yes)
     (property "Reference" "VIN" (at 85 46.19 0)
@@
     )
   )
-  (symbol (lib_id "Device:Q_PMOS_GSD") (at 120 50 0) (unit 1)
+  (symbol (lib_id "examples:MPMOS") (at 120 50 0) (unit 1)
     (in_bom yes) (on_board yes)
     (property "Reference" "MP1" (at 120 46.19 0)
@@
     )
   )
-  (symbol (lib_id "Device:Q_NMOS_GSD") (at 155 50 0) (unit 1)
+  (symbol (lib_id "examples:MNMOS") (at 155 50 0) (unit 1)
     (in_bom yes) (on_board yes)
     (property "Reference" "MN1" (at 155 46.19 0)
@@
     )
   )
-  (label "0" (at 50.00 54.50 0)
+  (symbol (lib_id "examples:GND") (at 44.00 50.00 0) (unit 1)
+    (in_bom yes) (on_board yes)
+    (property "Reference" "#PWR0001" (at 44.0 46.19 0)
+      (effects (font (size 1.27 1.27)) hide)
+    )
+    (property "Value" "GND" (at 44.0 53.81 0)
+      (effects (font (size 1.27 1.27)))
+    )
+    (property "Footprint" "" (at 0 0 0)
+      (effects (font (size 1.27 1.27)) hide)
+    )
+    (property "Datasheet" "" (at 0 0 0)
+      (effects (font (size 1.27 1.27)) hide)
+    )
+  )
+  (symbol (lib_id "examples:VCC") (at 32.00 38.00 0) (unit 1)
+    (in_bom yes) (on_board yes)
+    (property "Reference" "#PWR0002" (at 32.0 34.19 0)
+      (effects (font (size 1.27 1.27)) hide)
+    )
+    (property "Value" "VCC" (at 32.0 41.81 0)
+      (effects (font (size 1.27 1.27)))
+    )
+    (property "Footprint" "" (at 0 0 0)
+      (effects (font (size 1.27 1.27)) hide)
+    )
+    (property "Datasheet" "" (at 0 0 0)
+      (effects (font (size 1.27 1.27)) hide)
+    )
+  )
+  (label "GND" (at 38.00 48.50 0)
     (effects (font (size 1.27 1.27)) (justify left bottom))
   )
-  (wire (pts (xy 55.00 62.00) (xy 162.00 62.00))
+  (wire (pts (xy 43.00 60.80) (xy 162.00 60.80))
     (stroke (width 0) (type solid) (color 0 0 0 0))
   )
-  (wire (pts (xy 56.00 56.00) (xy 56.00 62.00))
+  (wire (pts (xy 56.00 56.00) (xy 56.00 60.80))
     (stroke (width 0) (type solid) (color 0 0 0 0))
   )
-  (junction (at 56.00 62.00) (diameter 1.016) (color 0 0 0 0))
-  (wire (pts (xy 91.00 56.00) (xy 91.00 62.00))
+  (junction (at 56.00 60.80) (diameter 1.016) (color 0 0 0 0))
+  (wire (pts (xy 91.00 56.00) (xy 91.00 60.80))
     (stroke (width 0) (type solid) (color 0 0 0 0))
   )
-  (junction (at 91.00 62.00) (diameter 1.016) (color 0 0 0 0))
-  (wire (pts (xy 157.00 56.00) (xy 157.00 62.00))
+  (junction (at 91.00 60.80) (diameter 1.016) (color 0 0 0 0))
+  (wire (pts (xy 157.00 56.00) (xy 157.00 60.80))
     (stroke (width 0) (type solid) (color 0 0 0 0))
   )
-  (junction (at 157.00 62.00) (diameter 1.016) (color 0 0 0 0))
-  (wire (pts (xy 161.00 56.00) (xy 161.00 62.00))
+  (junction (at 157.00 60.80) (diameter 1.016) (color 0 0 0 0))
+  (wire (pts (xy 161.00 56.00) (xy 161.00 60.80))
     (stroke (width 0) (type solid) (color 0 0 0 0))
   )
-  (junction (at 161.00 62.00) (diameter 1.016) (color 0 0 0 0))
-  (label "vdd" (at 38.00 41.00 0)
+  (junction (at 161.00 60.80) (diameter 1.016) (color 0 0 0 0))
+  (wire (pts (xy 44.00 50.00) (xy 44.00 60.80))
+    (stroke (width 0) (type solid) (color 0 0 0 0))
+  )
+  (junction (at 44.00 60.80) (diameter 1.016) (color 0 0 0 0))
+  (label "VCC" (at 26.00 35.00 0)
     (effects (font (size 1.27 1.27)) (justify left bottom))
   )
-  (wire (pts (xy 43.00 58.00) (xy 127.00 58.00))
+  (wire (pts (xy 31.00 54.50) (xy 127.00 54.50))
     (stroke (width 0) (type solid) (color 0 0 0 0))
   )
-  (wire (pts (xy 44.00 44.00) (xy 44.00 58.00))
+  (wire (pts (xy 44.00 44.00) (xy 44.00 54.50))
     (stroke (width 0) (type solid) (color 0 0 0 0))
   )
-  (junction (at 44.00 58.00) (diameter 1.016) (color 0 0 0 0))
-  (wire (pts (xy 122.00 56.00) (xy 122.00 58.00))
+  (junction (at 44.00 54.50) (diameter 1.016) (color 0 0 0 0))
+  (wire (pts (xy 122.00 56.00) (xy 122.00 54.50))
     (stroke (width 0) (type solid) (color 0 0 0 0))
   )
-  (junction (at 122.00 58.00) (diameter 1.016) (color 0 0 0 0))
-  (wire (pts (xy 126.00 56.00) (xy 126.00 58.00))
+  (junction (at 122.00 54.50) (diameter 1.016) (color 0 0 0 0))
+  (wire (pts (xy 126.00 56.00) (xy 126.00 54.50))
     (stroke (width 0) (type solid) (color 0 0 0 0))
   )
-  (junction (at 126.00 58.00) (diameter 1.016) (color 0 0 0 0))
+  (junction (at 126.00 54.50) (diameter 1.016) (color 0 0 0 0))
+  (wire (pts (xy 32.00 38.00) (xy 32.00 54.50))
+    (stroke (width 0) (type solid) (color 0 0 0 0))
+  )
+  (junction (at 32.00 54.50) (diameter 1.016) (color 0 0 0 0))
   (label "vin" (at 73.00 42.50 0)
     (effects (font (size 1.27 1.27)) (justify left bottom))
@@
     (path "/f4506daf-bd4d-5f0d-9ab2-7b9dab94c863" (reference "MP1") (unit 1) (value "PM1") (footprint ""))
     (path "/5f8db717-cf5d-5835-aecb-a1c06f647fe7" (reference "MN1") (unit 1) (value "NM1") (footprint ""))
+    (path "/b4802630-653f-5680-97fb-278aa6e5f6b5" (reference "#PWR0001") (unit 1) (value "GND") (footprint ""))
+    (path "/444c675b-9706-5ca9-bb39-d9f125d8e1c6" (reference "#PWR0002") (unit 1) (value "VCC") (footprint ""))
   )
 )
