File: examples/generated/kicad/opamp_inverting.kicad_sch (KiCad schematic)
At the start: 6 parts

Commit message: Generate schematics that are more intelligible and project structure that is closer to the KiCad demo behavior.
Other:
- note added: "pins 1:0 2:vminus 3:vout"
- note added: "pins 1:vcc 2:0"
- note added: "pins 1:vee 2:0"
- note added: "pins 1:vin 2:0"
- note added: "pins 1:vin 2:vminus"
- note added: "pins 1:vout 2:vminus"
Changed lines of the file:
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@@
     (effects (font (size 1.27 1.27)) (justify left))
+  )
+  (text "pins 1:vcc  2:0" (at 50 58 0)
+    (effects (font (size 1.0 1.0)) (justify left))
   )
   (symbol (lib_id "pspice:VSOURCE") (at 50 50 0) (unit 1)
@@
     (effects (font (size 1.27 1.27)) (justify left))
   )
+  (text "pins 1:vee  2:0" (at 85 58 0)
+    (effects (font (size 1.0 1.0)) (justify left))
+  )
   (symbol (lib_id "pspice:VSOURCE") (at 85 50 0) (unit 1)
     (in_bom yes) (on_board yes)
@@
   (text "nodes: vin 0" (at 120 42 0)
     (effects (font (size 1.27 1.27)) (justify left))
+  )
+  (text "pins 1:vin  2:0" (at 120 58 0)
+    (effects (font (size 1.0 1.0)) (justify left))
   )
   (symbol (lib_id "pspice:VSOURCE") (at 120 50 0) (unit 1)
@@
     (effects (font (size 1.27 1.27)) (justify left))
   )
+  (text "pins 1:vin  2:vminus" (at 155 58 0)
+    (effects (font (size 1.0 1.0)) (justify left))
+  )
   (symbol (lib_id "Device:R") (at 155 50 0) (unit 1)
     (in_bom yes) (on_board yes)
@@
   (text "nodes: vout vminus" (at 50 72 0)
     (effects (font (size 1.27 1.27)) (justify left))
+  )
+  (text "pins 1:vout  2:vminus" (at 50 88 0)
+    (effects (font (size 1.0 1.0)) (justify left))
   )
   (symbol (lib_id "Device:R") (at 50 80 0) (unit 1)
@@
     (effects (font (size 1.27 1.27)) (justify left))
   )
+  (text "pins 1:0  2:vminus  3:vout" (at 85 88 0)
+    (effects (font (size 1.0 1.0)) (justify left))
+  )
   (symbol (lib_id "Amplifier_Operational:LM358") (at 85 80 0) (unit 1)

Commit message: Attempt to clean up symbols and schematics to be more himan readable.
Other:
- note removed: "nodes: 0 vminus vout"
- note removed: "nodes: vcc 0"
- note removed: "nodes: vee 0"
- note removed: "nodes: vin 0"
- note removed: "nodes: vin vminus"
- note removed: "nodes: vout vminus"
- note removed: "pins 1:0 2:vminus 3:vout"
- note removed: "pins 1:vcc 2:0"
- note removed: "pins 1:vee 2:0"
- note removed: "pins 1:vin 2:0"
- note removed: "pins 1:vin 2:vminus"
- note removed: "pins 1:vout 2:vminus"
- title: (none) -> opamp_inverting
Changed lines of the file:
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@@
   (generator "mixedsig2cad")
   (paper "A4")
-  (text "nodes: vcc 0" (at 50 42 0)
-    (effects (font (size 1.27 1.27)) (justify left))
-  )
-  (text "pins 1:vcc  2:0" (at 50 58 0)
-    (effects (font (size 1.0 1.0)) (justify left))
+  (title_block
+    (title "opamp_inverting")
+    (date "2026-03-05")
+    (comment 1 "Generated by mixedsig2cad")
   )
   (symbol (lib_id "pspice:VSOURCE") (at 50 50 0) (unit 1)
@@
     )
   )
-  (text "nodes: vee 0" (at 85 42 0)
-    (effects (font (size 1.27 1.27)) (justify left))
-  )
-  (text "pins 1:vee  2:0" (at 85 58 0)
-    (effects (font (size 1.0 1.0)) (justify left))
-  )
   (symbol (lib_id "pspice:VSOURCE") (at 85 50 0) (unit 1)
     (in_bom yes) (on_board yes)
@@
       (effects (font (size 1.27 1.27)) hide)
     )
-  )
-  (text "nodes: vin 0" (at 120 42 0)
-    (effects (font (size 1.27 1.27)) (justify left))
-  )
-  (text "pins 1:vin  2:0" (at 120 58 0)
-    (effects (font (size 1.0 1.0)) (justify left))
   )
   (symbol (lib_id "pspice:VSOURCE") (at 120 50 0) (unit 1)
@@
     )
   )
-  (text "nodes: vin vminus" (at 155 42 0)
-    (effects (font (size 1.27 1.27)) (justify left))
-  )
-  (text "pins 1:vin  2:vminus" (at 155 58 0)
-    (effects (font (size 1.0 1.0)) (justify left))
-  )
   (symbol (lib_id "Device:R") (at 155 50 0) (unit 1)
     (in_bom yes) (on_board yes)
@@
       (effects (font (size 1.27 1.27)) hide)
     )
-  )
-  (text "nodes: vout vminus" (at 50 72 0)
-    (effects (font (size 1.27 1.27)) (justify left))
-  )
-  (text "pins 1:vout  2:vminus" (at 50 88 0)
-    (effects (font (size 1.0 1.0)) (justify left))
   )
   (symbol (lib_id "Device:R") (at 50 80 0) (unit 1)
@@
     )
   )
-  (text "nodes: 0 vminus vout" (at 85 72 0)
-    (effects (font (size 1.27 1.27)) (justify left))
-  )
-  (text "pins 1:0  2:vminus  3:vout" (at 85 88 0)
-    (effects (font (size 1.0 1.0)) (justify left))
-  )
   (symbol (lib_id "Amplifier_Operational:LM358") (at 85 80 0) (unit 1)
     (in_bom yes) (on_board yes)
@@
     )
   )
+  (label "0" (at 50.00 54.50 0)
+    (effects (font (size 1.27 1.27)) (justify left bottom))
+  )
+  (wire (pts (xy 55.00 66.50) (xy 127.00 66.50))
+    (stroke (width 0) (type solid) (color 0 0 0 0))
+  )
+  (wire (pts (xy 56.00 56.00) (xy 56.00 66.50))
+    (stroke (width 0) (type solid) (color 0 0 0 0))
+  )
+  (junction (at 56.00 66.50) (diameter 1.016) (color 0 0 0 0))
+  (wire (pts (xy 91.00 56.00) (xy 91.00 66.50))
+    (stroke (width 0) (type solid) (color 0 0 0 0))
+  )
+  (junction (at 91.00 66.50) (diameter 1.016) (color 0 0 0 0))
+  (wire (pts (xy 126.00 56.00) (xy 126.00 66.50))
+    (stroke (width 0) (type solid) (color 0 0 0 0))
+  )
+  (junction (at 126.00 66.50) (diameter 1.016) (color 0 0 0 0))
+  (wire (pts (xy 79.00 74.00) (xy 79.00 66.50))
+    (stroke (width 0) (type solid) (color 0 0 0 0))
+  )
+  (junction (at 79.00 66.50) (diameter 1.016) (color 0 0 0 0))
+  (label "vcc" (at 38.00 41.00 0)
+    (effects (font (size 1.27 1.27)) (justify left bottom))
+  )
+  (label "vee" (at 73.00 42.50 0)
+    (effects (font (size 1.27 1.27)) (justify left bottom))
+  )
+  (label "vin" (at 108.00 41.00 0)
+    (effects (font (size 1.27 1.27)) (justify left bottom))
+  )
+  (wire (pts (xy 114.00 44.00) (xy 149.00 44.00))
+    (stroke (width 0) (type solid) (color 0 0 0 0))
+  )
+  (label "vminus" (at 50.00 54.50 0)
+    (effects (font (size 1.27 1.27)) (justify left bottom))
+  )
+  (wire (pts (xy 55.00 78.00) (xy 162.00 78.00))
+    (stroke (width 0) (type solid) (color 0 0 0 0))
+  )
+  (wire (pts (xy 161.00 56.00) (xy 161.00 78.00))
+    (stroke (width 0) (type solid) (color 0 0 0 0))
+  )
+  (junction (at 161.00 78.00) (diameter 1.016) (color 0 0 0 0))
+  (wire (pts (xy 56.00 86.00) (xy 56.00 78.00))
+    (stroke (width 0) (type solid) (color 0 0 0 0))
+  )
+  (junction (at 56.00 78.00) (diameter 1.016) (color 0 0 0 0))
+  (wire (pts (xy 85.00 74.00) (xy 85.00 78.00))
+    (stroke (width 0) (type solid) (color 0 0 0 0))
+  )
+  (junction (at 85.00 78.00) (diameter 1.016) (color 0 0 0 0))
+  (label "vout" (at 38.00 71.00 0)
+    (effects (font (size 1.27 1.27)) (justify left bottom))
+  )
+  (wire (pts (xy 44.00 74.00) (xy 67.50 74.00))
+    (stroke (width 0) (type solid) (color 0 0 0 0))
+  )
+  (wire (pts (xy 67.50 74.00) (xy 67.50 86.00))
+    (stroke (width 0) (type solid) (color 0 0 0 0))
+  )
+  (wire (pts (xy 67.50 86.00) (xy 91.00 86.00))
+    (stroke (width 0) (type solid) (color 0 0 0 0))
+  )
+  (junction (at 67.50 74.00) (diameter 1.016) (color 0 0 0 0))
+  (junction (at 67.50 86.00) (diameter 1.016) (color 0 0 0 0))
   (sheet_instances
     (path "/" (page "1"))

Commit message: Attempt to add power symbology.
Parts:
- RF, RIN: symbol Device:R -> examples:R
- VCC, VEE, VIN: symbol pspice:VSOURCE -> examples:VSOURCE
- XU1: symbol Amplifier_Operational:LM358 -> examples:OPAMP
Changed lines of the file:
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@@
     (comment 1 "Generated by mixedsig2cad")
   )
-  (symbol (lib_id "pspice:VSOURCE") (at 50 50 0) (unit 1)
+  (symbol (lib_id "examples:VSOURCE") (at 50 50 0) (unit 1)
     (in_bom yes) (on_board yes)
     (property "Reference" "VCC" (at 50 46.19 0)
@@
     )
   )
-  (symbol (lib_id "pspice:VSOURCE") (at 85 50 0) (unit 1)
+  (symbol (lib_id "examples:VSOURCE") (at 85 50 0) (unit 1)
     (in_bom yes) (on_board yes)
     (property "Reference" "VEE" (at 85 46.19 0)
@@
     )
   )
-  (symbol (lib_id "pspice:VSOURCE") (at 120 50 0) (unit 1)
+  (symbol (lib_id "examples:VSOURCE") (at 120 50 0) (unit 1)
     (in_bom yes) (on_board yes)
     (property "Reference" "VIN" (at 120 46.19 0)
@@
     )
   )
-  (symbol (lib_id "Device:R") (at 155 50 0) (unit 1)
+  (symbol (lib_id "examples:R") (at 155 50 0) (unit 1)
     (in_bom yes) (on_board yes)
     (property "Reference" "RIN" (at 155 46.19 0)
@@
     )
   )
-  (symbol (lib_id "Device:R") (at 50 80 0) (unit 1)
+  (symbol (lib_id "examples:R") (at 50 80 0) (unit 1)
     (in_bom yes) (on_board yes)
     (property "Reference" "RF" (at 50 76.19 0)
@@
     )
   )
-  (symbol (lib_id "Amplifier_Operational:LM358") (at 85 80 0) (unit 1)
+  (symbol (lib_id "examples:OPAMP") (at 85 80 0) (unit 1)
     (in_bom yes) (on_board yes)
     (property "Reference" "XU1" (at 85 76.19 0)
@@
     )
   )
-  (label "0" (at 50.00 54.50 0)
-    (effects (font (size 1.27 1.27)) (justify left bottom))
-  )
-  (wire (pts (xy 55.00 66.50) (xy 127.00 66.50))
-    (stroke (width 0) (type solid) (color 0 0 0 0))
-  )
-  (wire (pts (xy 56.00 56.00) (xy 56.00 66.50))
-    (stroke (width 0) (type solid) (color 0 0 0 0))
-  )
-  (junction (at 56.00 66.50) (diameter 1.016) (color 0 0 0 0))
-  (wire (pts (xy 91.00 56.00) (xy 91.00 66.50))
-    (stroke (width 0) (type solid) (color 0 0 0 0))
-  )
-  (junction (at 91.00 66.50) (diameter 1.016) (color 0 0 0 0))
-  (wire (pts (xy 126.00 56.00) (xy 126.00 66.50))
-    (stroke (width 0) (type solid) (color 0 0 0 0))
-  )
-  (junction (at 126.00 66.50) (diameter 1.016) (color 0 0 0 0))
-  (wire (pts (xy 79.00 74.00) (xy 79.00 66.50))
-    (stroke (width 0) (type solid) (color 0 0 0 0))
-  )
-  (junction (at 79.00 66.50) (diameter 1.016) (color 0 0 0 0))
-  (label "vcc" (at 38.00 41.00 0)
-    (effects (font (size 1.27 1.27)) (justify left bottom))
-  )
+  (symbol (lib_id "examples:GND") (at 44.00 50.00 0) (unit 1)
+    (in_bom yes) (on_board yes)
+    (property "Reference" "#PWR0001" (at 44.0 46.19 0)
+      (effects (font (size 1.27 1.27)) hide)
+    )
+    (property "Value" "GND" (at 44.0 53.81 0)
+      (effects (font (size 1.27 1.27)))
+    )
+    (property "Footprint" "" (at 0 0 0)
+      (effects (font (size 1.27 1.27)) hide)
+    )
+    (property "Datasheet" "" (at 0 0 0)
+      (effects (font (size 1.27 1.27)) hide)
+    )
+  )
+  (symbol (lib_id "examples:VCC") (at 32.00 38.00 0) (unit 1)
+    (in_bom yes) (on_board yes)
+    (property "Reference" "#PWR0002" (at 32.0 34.19 0)
+      (effects (font (size 1.27 1.27)) hide)
+    )
+    (property "Value" "VCC" (at 32.0 41.81 0)
+      (effects (font (size 1.27 1.27)))
+    )
+    (property "Footprint" "" (at 0 0 0)
+      (effects (font (size 1.27 1.27)) hide)
+    )
+    (property "Datasheet" "" (at 0 0 0)
+      (effects (font (size 1.27 1.27)) hide)
+    )
+  )
+  (label "GND" (at 38.00 48.50 0)
+    (effects (font (size 1.27 1.27)) (justify left bottom))
+  )
+  (wire (pts (xy 43.00 64.40) (xy 127.00 64.40))
+    (stroke (width 0) (type solid) (color 0 0 0 0))
+  )
+  (wire (pts (xy 56.00 56.00) (xy 56.00 64.40))
+    (stroke (width 0) (type solid) (color 0 0 0 0))
+  )
+  (junction (at 56.00 64.40) (diameter 1.016) (color 0 0 0 0))
+  (wire (pts (xy 91.00 56.00) (xy 91.00 64.40))
+    (stroke (width 0) (type solid) (color 0 0 0 0))
+  )
+  (junction (at 91.00 64.40) (diameter 1.016) (color 0 0 0 0))
+  (wire (pts (xy 126.00 56.00) (xy 126.00 64.40))
+    (stroke (width 0) (type solid) (color 0 0 0 0))
+  )
+  (junction (at 126.00 64.40) (diameter 1.016) (color 0 0 0 0))
+  (wire (pts (xy 79.00 74.00) (xy 79.00 64.40))
+    (stroke (width 0) (type solid) (color 0 0 0 0))
+  )
+  (junction (at 79.00 64.40) (diameter 1.016) (color 0 0 0 0))
+  (wire (pts (xy 44.00 50.00) (xy 44.00 64.40))
+    (stroke (width 0) (type solid) (color 0 0 0 0))
+  )
+  (junction (at 44.00 64.40) (diameter 1.016) (color 0 0 0 0))
+  (label "VCC" (at 26.00 35.00 0)
+    (effects (font (size 1.27 1.27)) (justify left bottom))
+  )
+  (wire (pts (xy 44.00 44.00) (xy 38.00 44.00))
+    (stroke (width 0) (type solid) (color 0 0 0 0))
+  )
+  (wire (pts (xy 38.00 44.00) (xy 38.00 38.00))
+    (stroke (width 0) (type solid) (color 0 0 0 0))
+  )
+  (wire (pts (xy 38.00 38.00) (xy 32.00 38.00))
+    (stroke (width 0) (type solid) (color 0 0 0 0))
+  )
+  (junction (at 38.00 44.00) (diameter 1.016) (color 0 0 0 0))
+  (junction (at 38.00 38.00) (diameter 1.016) (color 0 0 0 0))
   (label "vee" (at 73.00 42.50 0)
     (effects (font (size 1.27 1.27)) (justify left bottom))
@@
     (path "/2af704cc-8e18-5163-a150-531370848bee" (reference "RF") (unit 1) (value "100k") (footprint ""))
     (path "/14787423-abe0-5cea-9c2c-1b908a510b95" (reference "XU1") (unit 1) (value "OPAMP") (footprint ""))
+    (path "/99d184dd-c08a-5bc9-86ea-1c4b84e15058" (reference "#PWR0001") (unit 1) (value "GND") (footprint ""))
+    (path "/7b569932-0d2f-5759-bd01-500895a432c5" (reference "#PWR0002") (unit 1) (value "VCC") (footprint ""))
   )
 )
