File: examples/generated/kicad/rc_lowpass.kicad_sch (KiCad schematic)
At the start: 3 parts

Commit message: Generate schematics that are more intelligible and project structure that is closer to the KiCad demo behavior.
Other:
- note added: "pins 1:vin 2:0"
- note added: "pins 1:vin 2:vout"
- note added: "pins 1:vout 2:0"
Changed lines of the file:
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@@
     (effects (font (size 1.27 1.27)) (justify left))
+  )
+  (text "pins 1:vin  2:0" (at 50 58 0)
+    (effects (font (size 1.0 1.0)) (justify left))
   )
   (symbol (lib_id "pspice:VSOURCE") (at 50 50 0) (unit 1)
@@
     (effects (font (size 1.27 1.27)) (justify left))
   )
+  (text "pins 1:vin  2:vout" (at 85 58 0)
+    (effects (font (size 1.0 1.0)) (justify left))
+  )
   (symbol (lib_id "Device:R") (at 85 50 0) (unit 1)
     (in_bom yes) (on_board yes)
@@
     (effects (font (size 1.27 1.27)) (justify left))
   )
+  (text "pins 1:vout  2:0" (at 120 58 0)
+    (effects (font (size 1.0 1.0)) (justify left))
+  )
   (symbol (lib_id "Device:C") (at 120 50 0) (unit 1)

Commit message: Attempt to clean up symbols and schematics to be more himan readable.
Other:
- note removed: "nodes: vin 0"
- note removed: "nodes: vin vout"
- note removed: "nodes: vout 0"
- note removed: "pins 1:vin 2:0"
- note removed: "pins 1:vin 2:vout"
- note removed: "pins 1:vout 2:0"
- title: (none) -> rc_lowpass
Changed lines of the file:
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@@
   (generator "mixedsig2cad")
   (paper "A4")
-  (text "nodes: vin 0" (at 50 42 0)
-    (effects (font (size 1.27 1.27)) (justify left))
-  )
-  (text "pins 1:vin  2:0" (at 50 58 0)
-    (effects (font (size 1.0 1.0)) (justify left))
+  (title_block
+    (title "rc_lowpass")
+    (date "2026-03-05")
+    (comment 1 "Generated by mixedsig2cad")
   )
   (symbol (lib_id "pspice:VSOURCE") (at 50 50 0) (unit 1)
@@
     )
   )
-  (text "nodes: vin vout" (at 85 42 0)
-    (effects (font (size 1.27 1.27)) (justify left))
-  )
-  (text "pins 1:vin  2:vout" (at 85 58 0)
-    (effects (font (size 1.0 1.0)) (justify left))
-  )
   (symbol (lib_id "Device:R") (at 85 50 0) (unit 1)
     (in_bom yes) (on_board yes)
@@
       (effects (font (size 1.27 1.27)) hide)
     )
-  )
-  (text "nodes: vout 0" (at 120 42 0)
-    (effects (font (size 1.27 1.27)) (justify left))
-  )
-  (text "pins 1:vout  2:0" (at 120 58 0)
-    (effects (font (size 1.0 1.0)) (justify left))
   )
   (symbol (lib_id "Device:C") (at 120 50 0) (unit 1)
@@
     )
   )
+  (label "0" (at 50.00 54.50 0)
+    (effects (font (size 1.27 1.27)) (justify left bottom))
+  )
+  (wire (pts (xy 56.00 56.00) (xy 126.00 56.00))
+    (stroke (width 0) (type solid) (color 0 0 0 0))
+  )
+  (label "vin" (at 38.00 41.00 0)
+    (effects (font (size 1.27 1.27)) (justify left bottom))
+  )
+  (wire (pts (xy 44.00 44.00) (xy 79.00 44.00))
+    (stroke (width 0) (type solid) (color 0 0 0 0))
+  )
+  (label "vout" (at 85.00 42.50 0)
+    (effects (font (size 1.27 1.27)) (justify left bottom))
+  )
+  (wire (pts (xy 91.00 56.00) (xy 102.50 56.00))
+    (stroke (width 0) (type solid) (color 0 0 0 0))
+  )
+  (wire (pts (xy 102.50 56.00) (xy 102.50 44.00))
+    (stroke (width 0) (type solid) (color 0 0 0 0))
+  )
+  (wire (pts (xy 102.50 44.00) (xy 114.00 44.00))
+    (stroke (width 0) (type solid) (color 0 0 0 0))
+  )
+  (junction (at 102.50 56.00) (diameter 1.016) (color 0 0 0 0))
+  (junction (at 102.50 44.00) (diameter 1.016) (color 0 0 0 0))
   (sheet_instances
     (path "/" (page "1"))

Commit message: Attempt to add power symbology.
Parts:
- C1: symbol Device:C -> examples:CAP
- R1: symbol Device:R -> examples:R
- V1: symbol pspice:VSOURCE -> examples:VSOURCE
Changed lines of the file:
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@@
     (comment 1 "Generated by mixedsig2cad")
   )
-  (symbol (lib_id "pspice:VSOURCE") (at 50 50 0) (unit 1)
+  (symbol (lib_id "examples:VSOURCE") (at 50 50 0) (unit 1)
     (in_bom yes) (on_board yes)
     (property "Reference" "V1" (at 50 46.19 0)
@@
     )
   )
-  (symbol (lib_id "Device:R") (at 85 50 0) (unit 1)
+  (symbol (lib_id "examples:R") (at 85 50 0) (unit 1)
     (in_bom yes) (on_board yes)
     (property "Reference" "R1" (at 85 46.19 0)
@@
     )
   )
-  (symbol (lib_id "Device:C") (at 120 50 0) (unit 1)
+  (symbol (lib_id "examples:CAP") (at 120 50 0) (unit 1)
     (in_bom yes) (on_board yes)
     (property "Reference" "C1" (at 120 46.19 0)
@@
     )
   )
-  (label "0" (at 50.00 54.50 0)
+  (symbol (lib_id "examples:GND") (at 44.00 50.00 0) (unit 1)
+    (in_bom yes) (on_board yes)
+    (property "Reference" "#PWR0001" (at 44.0 46.19 0)
+      (effects (font (size 1.27 1.27)) hide)
+    )
+    (property "Value" "GND" (at 44.0 53.81 0)
+      (effects (font (size 1.27 1.27)))
+    )
+    (property "Footprint" "" (at 0 0 0)
+      (effects (font (size 1.27 1.27)) hide)
+    )
+    (property "Datasheet" "" (at 0 0 0)
+      (effects (font (size 1.27 1.27)) hide)
+    )
+  )
+  (label "GND" (at 38.00 48.50 0)
     (effects (font (size 1.27 1.27)) (justify left bottom))
   )
-  (wire (pts (xy 56.00 56.00) (xy 126.00 56.00))
+  (wire (pts (xy 43.00 60.00) (xy 127.00 60.00))
     (stroke (width 0) (type solid) (color 0 0 0 0))
   )
+  (wire (pts (xy 56.00 56.00) (xy 56.00 60.00))
+    (stroke (width 0) (type solid) (color 0 0 0 0))
+  )
+  (junction (at 56.00 60.00) (diameter 1.016) (color 0 0 0 0))
+  (wire (pts (xy 126.00 56.00) (xy 126.00 60.00))
+    (stroke (width 0) (type solid) (color 0 0 0 0))
+  )
+  (junction (at 126.00 60.00) (diameter 1.016) (color 0 0 0 0))
+  (wire (pts (xy 44.00 50.00) (xy 44.00 60.00))
+    (stroke (width 0) (type solid) (color 0 0 0 0))
+  )
+  (junction (at 44.00 60.00) (diameter 1.016) (color 0 0 0 0))
   (label "vin" (at 38.00 41.00 0)
     (effects (font (size 1.27 1.27)) (justify left bottom))
@@
     (path "/f9364b86-dfb1-51e8-9247-72a2484cf109" (reference "R1") (unit 1) (value "1k") (footprint ""))
     (path "/fff04eb7-92e3-5e3e-9950-c8b8ac3c6096" (reference "C1") (unit 1) (value "100n") (footprint ""))
+    (path "/4d746a25-6e32-5362-9bf4-cd3363ff6631" (reference "#PWR0001") (unit 1) (value "GND") (footprint ""))
   )
 )
